File: FoxHuntAttenuator.kicad_pcb (KiCad board)
At the start: 2 copper layers, 187.2 x 36.6 mm, 38 parts, among them J1 Conn_Coaxial, J2 Conn_Coaxial, SW1 SW_SPST, SW2 SW_SPST, SW3 SW_SPST, SW4 SW_SPST, SW5 SW_SPST, SW6 SW_SPST, SW7 SW_SPST, SW8 SW_SPST

Commit message: pcb routing
Parts:
- moved R6 12.7 mm to (122.9, 111.0), turned to 180 degrees
Routing:
- net Net-(SW2-B): track 0.00 -> 69.2 mm
- net Net-(SW3-B): track 0.00 -> 62.0 mm
- net Net-(SW5-B): track 0.00 -> 57.9 mm
- net Net-(SW4-B): track 0.00 -> 57.7 mm
- net Net-(SW7-B): track 0.00 -> 56.7 mm
- net Net-(SW6-B): track 0.00 -> 56.4 mm
- net Net-(SW1-B): track 0.00 -> 53.3 mm
- net Net-(J2-In): track 0.00 -> 37.8 mm
- net Net-(J1-In): track 0.00 -> 29.1 mm
- added copper zone on B.Cu, net GND

Commit message: updating pcb
Parts:
- moved R9 18.8 mm to (141.7, 111.0)
- moved R7 18.8 mm to (141.7, 129.8)
- moved R11 12.7 mm to (144.8, 126.8), turned to 90 degrees
- moved R5 12.7 mm to (107.2, 126.8), turned to 90 degrees
Routing:
- net Net-(SW2-B): track 69.2 -> 55.3 mm
- net Net-(SW3-B): track 62.0 -> 56.6 mm
- net Net-(SW1-B): track 53.3 -> 48.9 mm
- net Net-(SW4-B): track 57.7 -> 56.5 mm
Other:
- board text added: "0-144dB Attenuation. Each toggle on will give an additional 18dB of attenuation."
- board text added: "FOXHUNT PI ATTENUATOR NETWORK"
