File: FoxHuntAttenuator.kicad_pcb (KiCad board)
At the start: 2 copper layers, 187.2 x 36.6 mm, 38 parts, among them J1 Conn_Coaxial, J2 Conn_Coaxial, SW1 SW_SPST, SW2 SW_SPST, SW3 SW_SPST, SW4 SW_SPST, SW5 SW_SPST, SW6 SW_SPST, SW7 SW_SPST, SW8 SW_SPST

Commit message: finishing pcb layout
Parts:
- moved H4 2.94 mm to (73.1, 105.4)
- moved H3 2.80 mm to (73.1, 135.4)
- moved H1 2.43 mm to (253.8, 105.4)
- moved H2 2.39 mm to (253.8, 135.4)
Changed lines of the file:
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@@
 	(footprint "MountingHole:MountingHole_2.7mm_M2.5"
 		(layer "F.Cu")
-		(at 252.476 107.442)
+		(at 253.8 105.4)
 		(descr "Mounting Hole 2.7mm, no annular, M2.5")
 		(tags "mounting hole 2.7mm no annular m2.5")
@@
 	(footprint "MountingHole:MountingHole_2.7mm_M2.5"
 		(layer "F.Cu")
-		(at 252.222 133.604)
+		(at 253.8 135.4)
 		(descr "Mounting Hole 2.7mm, no annular, M2.5")
 		(tags "mounting hole 2.7mm no annular m2.5")
@@
 	(footprint "MountingHole:MountingHole_2.7mm_M2.5"
 		(layer "F.Cu")
-		(at 75.438 133.858)
+		(at 73.1 135.4)
 		(descr "Mounting Hole 2.7mm, no annular, M2.5")
 		(tags "mounting hole 2.7mm no annular m2.5")
@@
 	(footprint "MountingHole:MountingHole_2.7mm_M2.5"
 		(layer "F.Cu")
-		(at 75.438 107.188)
+		(at 73.1 105.4)
 		(descr "Mounting Hole 2.7mm, no annular, M2.5")
 		(tags "mounting hole 2.7mm no annular m2.5")
