File: FoxHuntAttenuator.kicad_sch (KiCad schematic)
At the start: 34 parts, among them J1 Conn_Coaxial, J2 Conn_Coaxial, SW1 SW_SPST, SW2 SW_SPST, SW3 SW_SPST, SW4 SW_SPST, SW5 SW_SPST, SW6 SW_SPST, SW7 SW_SPST, SW8 SW_SPST

Commit message: pcb layout
Parts:
- added H1, H2, H3, H4: MountingHole, MountingHole:MountingHole_2.7mm_M2.5, symbol Mechanical:MountingHole
